File: ZX_BUS_Mouse.kicad_pcb (KiCad board)
At the start: 2 copper layers, 99.1 x 40 mm, 28 parts, among them J1 X1A, J2 X1B, J4 Mini-DIN-6, J5 Conn_02x03_Odd_Even ISP, J6 Conn_01x04 Debug, J7 Conn_02x05_Odd_Even JTAG, U1 ATmega8A-A, U2 EPM3032ALC44, U3 AMS1117-3.3

Commit message: Rename libs/my_lib.pretty libs/zx_bus.pretty.
Parts:
- J1, J2: footprint my_lib:PinSocket_1x31_P2.54mm_2 -> zx_bus:PinSocket_1x31_P2.54mm_2
Changed lines of the file:
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@@
     )
   )
-  (footprint "my_lib:PinSocket_1x31_P2.54mm_2" (layer "F.Cu")
+  (footprint "zx_bus:PinSocket_1x31_P2.54mm_2" (layer "F.Cu")
     (at 53.975 145.034 90)
     (descr "Through hole straight socket strip, 1x31, 2.54mm pitch, single row (from Kicad 4.0.7), script generated")
@@
     )
   )
-  (footprint "my_lib:PinSocket_1x31_P2.54mm_2" (layer "B.Cu")
+  (footprint "zx_bus:PinSocket_1x31_P2.54mm_2" (layer "B.Cu")
     (at 53.975 145.034 -90)
     (descr "Through hole straight socket strip, 1x31, 2.54mm pitch, single row (from Kicad 4.0.7), script generated")
