File: KiCad/ZX_BUS_Mouse.kicad_sch (KiCad schematic)
At the start: 28 parts, among them J1 X1A, J2 X1B, J4 Mini-DIN-6, J5 Conn_02x03_Odd_Even ISP, J6 Conn_01x04 Debug, J7 Conn_02x05_Odd_Even JTAG, U1 ATmega8A-A, U2 EPM3032ALC44, U3 AMS1117-3.3

Commit message: Add 74LVC1G125DB 3-state buffer for IORQGE/IOGE signal: 5V output signal level. Resolve issue with ZX-BUS XTRaiser, prevent potential issues with 5V IORQGE back current from other cards to CPLD output pin. Change CPLD IORQGE output logic to 2-state. Swap D3/D4 CPLD pins.
Parts:
- added U4: 74LVC1G125DB, Package_TO_SOT_SMD:SOT-23-5_HandSoldering, symbol 74xGxx:74LVC1G125
Connections:
- net *D3: now also U2.21 (A16); no longer U2.18 (A13)
- net *D4: now also U2.18 (A13); no longer U2.21 (A16)
- net GND: now also U4.3 (GND)
- net IOGE/: now also U4.4; no longer U2.20 (A15)
- net VCC: now also U4.2, U4.5 (VCC)
- new net IORQGE/: U2.20 (A15), U4.1
Changed lines of the file:
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@@
+    (stroke (width 0) (type default))
+  )
+  (wire (pts (xy 203.581 118.745) (xy 213.36 118.745))
     (stroke (width 0) (type default))
   )
@@
   )
   (wire (pts (xy 60.96 25.4) (xy 60.96 26.67))
+    (stroke (width 0) (type default))
+  )
+  (wire (pts (xy 216.281 128.905) (xy 222.758 128.905))
     (stroke (width 0) (type default))
   )
@@
     (effects (font (size 1.27 1.27)) (justify left bottom))
   )
+  (label "IOGE{slash}" (at 216.662 128.905 0) (fields_autoplaced)
+    (effects (font (size 1.27 1.27)) (justify left bottom))
+  )
   (label "TDO" (at 158.75 96.52 0) (fields_autoplaced)
     (effects (font (size 1.27 1.27)) (justify left bottom))
@@
     (effects (font (size 1.27 1.27)) (justify left bottom))
   )
-  (label "*D3" (at 133.35 58.42 0) (fields_autoplaced)
+  (label "*D4" (at 133.35 58.42 0) (fields_autoplaced)
     (effects (font (size 1.27 1.27)) (justify left bottom))
   )
@@
     (effects (font (size 1.27 1.27)) (justify left bottom))
   )
+  (label "IORQGE{slash}" (at 204.47 118.745 0) (fields_autoplaced)
+    (effects (font (size 1.27 1.27)) (justify left bottom))
+  )
   (label "*A0" (at 189.23 45.72 0) (fields_autoplaced)
     (effects (font (size 1.27 1.27)) (justify left bottom))
@@
     (effects (font (size 1.27 1.27)) (justify left bottom))
   )
-  (label "IOGE{slash}" (at 130.81 63.5 0) (fields_autoplaced)
+  (label "IORQGE{slash}" (at 129.54 63.5 0) (fields_autoplaced)
     (effects (font (size 1.27 1.27)) (justify left bottom))
   )
@@
     (effects (font (size 1.27 1.27)) (justify left bottom))
   )
-  (label "*D4" (at 133.35 66.04 0) (fields_autoplaced)
+  (label "*D3" (at 133.35 66.04 0) (fields_autoplaced)
     (effects (font (size 1.27 1.27)) (justify left bottom))
   )
@@
     )
   )
+  (symbol (lib_id "power:VCC") (at 198.501 118.745 0) (unit 1)
+    (in_bom yes) (on_board yes) (dnp no) (fields_autoplaced)
+    (property "Reference" "#PWR023" (at 198.501 122.555 0)
+      (effects (font (size 1.27 1.27)) hide)
+    )
+    (property "Value" "VCC" (at 198.501 114.173 0)
+      (effects (font (size 1.27 1.27)))
+    )
+    (property "Footprint" "" (at 198.501 118.745 0)
+      (effects (font (size 1.27 1.27)) hide)
+    )
+    (property "Datasheet" "" (at 198.501 118.745 0)
+      (effects (font (size 1.27 1.27)) hide)
+    )
+    (pin "1")
+    (instances
+      (project "ZX_BUS_Mouse"
+        (path "/3450efc4-f02c-4d95-a19b-bf60e75dcf1f"
+          (reference "#PWR023") (unit 1)
+        )
+      )
+    )
+  )
   (symbol (lib_id "power:GND") (at 60.96 104.14 0) (unit 1)
     (in_bom yes) (on_board yes) (dnp no) (fields_autoplaced)
@@
     )
   )
+  (symbol (lib_id "power:VCC") (at 188.341 128.905 90) (unit 1)
+    (in_bom yes) (on_board yes) (dnp no) (fields_autoplaced)
+    (property "Reference" "#PWR024" (at 192.151 128.905 0)
+      (effects (font (size 1.27 1.27)) hide)
+    )
+    (property "Value" "VCC" (at 184.531 128.905 90)
+      (effects (font (size 1.27 1.27)) (justify left))
+    )
+    (property "Footprint" "" (at 188.341 128.905 0)
+      (effects (font (size 1.27 1.27)) hide)
+    )
+    (property "Datasheet" "" (at 188.341 128.905 0)
+      (effects (font (size 1.27 1.27)) hide)
+    )
+    (pin "1")
+    (instances
+      (project "ZX_BUS_Mouse"
+        (path "/3450efc4-f02c-4d95-a19b-bf60e75dcf1f"
+          (reference "#PWR024") (unit 1)
+        )
+      )
+    )
+  )
   (symbol (lib_id "power:GND") (at 147.32 148.59 0) (unit 1)
     (in_bom yes) (on_board yes) (dnp no) (fields_autoplaced)
@@
         )
       )
+    )
+  )
+  (symbol (lib_id "power:GND") (at 198.501 139.065 0) (unit 1)
+    (in_bom yes) (on_board yes) (dnp no) (fields_autoplaced)
+    (property "Reference" "#PWR022" (at 198.501 145.415 0)
+      (effects (font (size 1.27 1.27)) hide)
+    )
+    (property "Value" "GND" (at 198.501 144.399 0)
+      (effects (font (size 1.27 1.27)))
+    )
+    (property "Footprint" "" (at 198.501 139.065 0)
+      (effects (font (size 1.27 1.27)) hide)
+    )
+    (property "Datasheet" "" (at 198.501 139.065 0)
+      (effects (font (size 1.27 1.27)) hide)
+    )
+    (pin "1")
+    (instances
+      (project "ZX_BUS_Mouse"
+        (path "/3450efc4-f02c-4d95-a19b-bf60e75dcf1f"
+          (reference "#PWR022") (unit 1)
+        )
+      )
+    )
+  )
+  (symbol (lib_id "74xGxx:74LVC1G125") (at 203.581 128.905 0) (unit 1)
+    (in_bom yes) (on_board yes) (dnp no)
+    (property "Reference" "U4" (at 209.423 135.128 0)
+      (effects (font (size 1.27 1.27)))
+    )
+    (property "Value" "74LVC1G125DB" (at 209.423 137.668 0)
+      (effects (font (size 1.27 1.27)))
+    )
+    (property "Footprint" "Package_TO_SOT_SMD:SOT-23-5_HandSoldering" (at 203.581 147.955 0)
+      (effects (font (size 1.27 1.27)) hide)
+    )
+    (property "Datasheet" "https://www.ti.com/lit/ds/symlink/sn74lvc1g125.pdf" (at 203.581 128.905 0)
+      (effects (font (size 1.27 1.27)) hide)
+    )
+    (pin "4")
+    (pin "1")
+    (pin "5")
+    (pin "3")
+    (pin "2")
+    (instances
+      (project "ZX_BUS_Mouse"
+        (path "/3450efc4-f02c-4d95-a19b-bf60e75dcf1f"
+          (reference "U4") (unit 1)
+        )
+      )

Commit message: Add external PS/2 mouse bracket connector (common 486-Pentium AT motherboards pinout). Add debug UART connector (RX/TX). Move I2C debug connector, move optional R8, R9 pullup resistors to backside. Change Mini DIN connector drill holes diameter from 0.8 to 0.9 mm. Alter silkscreen labels.
Parts:
- added J3: UART, Connector_PinHeader_2.54mm:PinHeader_1x02_P2.54mm_Vertical, symbol Connector_Generic:Conn_01x02
- added J8: PS/2 External Bracket, Connector_PinHeader_2.54mm:PinHeader_2x04_P2.54mm_Vertical, symbol Connector_Generic:Conn_02x04_Odd_Even
- J5: value Conn_02x03_Odd_Even ISP -> ISP
- J6: value Conn_01x04 Debug -> Debug
- J7: value Conn_02x05_Odd_Even JTAG -> JTAG
Connections:
- net GND: now also J8.7 (Pin_7)
- net MCLK: now also J8.8 (Pin_8)
- net MDAT: now also J8.5 (Pin_5)
- net VCC: now also J8.1 (Pin_1)
- net RX: now reaches U1.30 (PD0)
- net RX: now also J3.1 (Pin_1)
- net TX: now reaches U1.31 (PD1)
- net TX: now also J3.2 (Pin_2)
- no-connect marks 53 -> 55
Other:
- note removed: "IO?"
- moved on the sheet: R2, R3
